File: eagle/Wheels heaters/Control.sch (EAGLE design)
At the start: 53 parts, among them IC1 LD1117, IC2 74LS47N, IC3 74LS47N, Q1 16MHz, SW1 AYZ0202, T1 2N7002, T2 2N7002, U1 ATMEGA168#

Commit message: Update Control.sch
Other:
- note added: "Wheel heaters & thermistors"
- note removed: "Wheel heaters & termistors"
Changed lines of the file:
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@@
 <wire x1="-116.84" y1="78.74" x2="-2.54" y2="78.74" width="0.1524" layer="97" style="shortdash"/>
 <text x="-116.84" y="78.74" size="1.778" layer="97">Displays &amp; leds</text>
-<text x="2.54" y="22.86" size="1.778" layer="97">Wheel heaters &amp; termistors</text>
+<text x="2.54" y="22.86" size="1.778" layer="97">Wheel heaters &amp; thermistors</text>
 <wire x1="2.54" y1="22.86" x2="2.54" y2="-22.86" width="0.1524" layer="97" style="shortdash"/>
 <wire x1="2.54" y1="-22.86" x2="127" y2="-22.86" width="0.1524" layer="97" style="shortdash"/>
